Commit message: Built the great wall of gazebo

File: workspace/limo_simulation/urdf/limo_four_diff.xacro (robot description, xacro)
@@ -64,3 +64,7 @@
         <origin xyz="${-wheelbase/2} ${-track/2} ${wheel_vertical_offset}" rpy="${M_PI} 0 0" />
     </xacro:limo_wheel>
+    <!-- LiDAR sensor -->
+    <xacro:limo_laser parent_prefix="base_link" frame_prefix="laser">
+        <origin xyz="0.0 0.0 0.08" rpy="0 0 0"/>
+    </xacro:limo_laser>
 </robot>
